File: telemetry-rusolar.kicad_sch (KiCad schematic)
At the start: 50 parts, among them J1 USART2, J10 Conn_01x16_Socket, J11 Conn_01x16_Socket, J12 Conn_02x16_Odd_Even, J13 Conn_02x16_Odd_Even, J14 Conn_01x16_Socket, J15 Conn_01x16_Socket, J2 USB_B_Micro, J4 SPI1, J5 SWD, J6 I2C1, J9 Micro_SD_Card, SW1 RESET, SW2 SW_BOOT, U2 STM32H723ZGTx, Y1 50MHz

Commit message: Changed schematics
Parts:
- removed C25, C26: 100n, symbol Device:C
- removed C27: 10u, symbol Device:C
- removed J15: Conn_01x16_Socket, symbol Connector:Conn_01x16_Socket
- removed J2: USB_B_Micro, symbol Connector:USB_B_Micro
- removed J9: Micro_SD_Card, symbol Connector:Micro_SD_Card
- removed R10, R11, R12, R13, R14, R9: 47k, symbol Device:R
- added C28: 100n, symbol Device:C
- added C29: 10u, symbol Device:C
- added J16: USB_C_Receptacle_USB2.0_14P, symbol Connector:USB_C_Receptacle_USB2.0_14P
- added J17: Micro_SD_Card, symbol Connector:Micro_SD_Card
- added J18: Conn_01x10_Socket, symbol Connector:Conn_01x10_Socket
- added J2, J9: Conn_01x16_Socket, symbol Connector:Conn_01x16_Socket
- added R15, R16, R17, R18, R19: 47k, symbol Device:R
- added R2, R7: 5k1, symbol Device:R
- C21, C22: value C -> 14p
- renumbered NOTE_SW to NOTE_SW1
Connections:
- net +3.3V: now also J17.4 (VDD), R15.2, R16.2, R17.2, R18.2, R19.2
- net GND: now also C29.2, J16.A1 (GND), J16.A12 (GND), J16.B1 (GND), J16.B12 (GND), J16.S1 (SHIELD), J17.6 (VSS), J17.9 (SHIELD), R2.2, R7.2
- net SD1_CK: now also J17.5 (CLK)
- net SD1_CMD: now also C28.1, J17.3 (CMD), R19.1
- net SD1_D0: now also J17.7 (DAT0), R15.1
- net SD1_D1: now also J17.8 (DAT1), R18.1
- net SD1_D2: now also J17.1 (DAT2), R17.1
- net SD1_D3: now also J17.2 (DAT3/CD), R16.1
- net USB_D+: now also J16.A6 (D+), J16.B6 (D+)
- net USB_D-: now also J16.A7 (D-), J16.B7 (D-)
- net VBUS: now also J16.A4 (VBUS), J16.A9 (VBUS), J16.B4 (VBUS), J16.B9 (VBUS)
- net PE2: now reaches J14.14 (Pin_14), U2.1 (PE2)
- net PF0: now reaches J11.16 (Pin_16), U2.10 (PF0)
- net PA8: now reaches U2.100 (PA8)
- net PA8: now also J2.4 (Pin_4)
- net PA9: now reaches U2.101 (PA9)
- net PA9: now also J2.5 (Pin_5)
- net PA10: now reaches U2.102 (PA10)
- net PA10: now also J2.6 (Pin_6)
- net PF1: now reaches J11.15 (Pin_15), U2.11 (PF1)
- net PA15: now reaches U2.110 (PA15(JTDI))
- net PA15: now also J2.7 (Pin_7)
- net PD3: now reaches U2.117 (PD3)
- net PD3: now also J9.14 (Pin_14)
- net PD4: now reaches U2.118 (PD4)
- net PD4: now also J9.15 (Pin_15)
- net PD5: now reaches U2.119 (PD5)
- net PD5: now also J9.16 (Pin_16)
- net PF2: now reaches J11.14 (Pin_14), U2.12 (PF2)
- net PD6: now reaches U2.122 (PD6)
- net PD6: now also J18.1 (Pin_1)
- net PD7: now reaches U2.123 (PD7)
- net PD7: now also J18.2 (Pin_2)
- net PF3: now reaches J11.13 (Pin_13), U2.13 (PF3)
- net PB4: now reaches U2.134 (PB4(NJTRST))
- net PB4: now also J2.11 (Pin_11)
- net PB5: now reaches U2.135 (PB5)
- net PB5: now also J2.12 (Pin_12)
- net PB8: now reaches U2.139 (PB8)
- net PB8: now also J2.13 (Pin_13)
- net PF4: now reaches J11.12 (Pin_12), U2.14 (PF4)
- net PB9: now reaches U2.140 (PB9)
- net PB9: now also J2.14 (Pin_14)
- net PE0: now reaches J14.16 (Pin_16), U2.141 (PE0)
- net PE1: now reaches J14.15 (Pin_15), U2.142 (PE1)
- net PF5: now reaches J11.11 (Pin_11), U2.15 (PF5)
- net PF6: now reaches J11.10 (Pin_10), U2.18 (PF6)
- net PF7: now reaches J11.9 (Pin_9), U2.19 (PF7)
- net PE3: now reaches J14.13 (Pin_13), U2.2 (PE3)
- net PF8: now reaches J11.8 (Pin_8), U2.20 (PF8)
- net PF9: now reaches J11.7 (Pin_7), U2.21 (PF9)
- net PF10: now reaches J11.6 (Pin_6), U2.22 (PF10)
- net PC0: now reaches U2.26 (PC0)
- net PC0: now also J9.2 (Pin_2)
- net PC1: now reaches U2.27 (PC1)
- net PC1: now also J9.3 (Pin_3)
- net PC2_C: now reaches U2.28 (PC2_C)
- net PC2_C: now also J9.4 (Pin_4)
- net PC3_C: now reaches U2.29 (PC3_C)
- net PC3_C: now also J9.5 (Pin_5)
- net PE4: now reaches J14.12 (Pin_12), U2.3 (PE4)
- net PA0: now reaches U2.34 (PA0)
- net PA0: now also J2.1 (Pin_1)
- net PA1: now reaches U2.35 (PA1)
- net PA1: now also J2.2 (Pin_2)
- net PE5: now reaches J14.11 (Pin_11), U2.4 (PE5)
- net PA4: now reaches U2.40 (PA4)
- net PA4: now also J2.3 (Pin_3)
- net PC4: now reaches U2.44 (PC4)
- net PC4: now also J9.6 (Pin_6)
- net PC5: now reaches U2.45 (PC5)
- net PC5: now also J9.7 (Pin_7)
- net PB0: now reaches U2.46 (PB0)
- net PB0: now also J2.8 (Pin_8)
- net PB1: now reaches U2.47 (PB1)
- net PB1: now also J2.9 (Pin_9)
- net PB2: now reaches U2.48 (PB2)
- net PB2: now also J2.10 (Pin_10)
- net PF11: now reaches J11.5 (Pin_5), U2.49 (PF11)
- net PE6: now reaches J14.10 (Pin_10), U2.5 (PE6)
- net PF12: now reaches J11.4 (Pin_4), U2.50 (PF12)
- net PF13: now reaches J11.3 (Pin_3), U2.53 (PF13)
- net PF14: now reaches J11.2 (Pin_2), U2.54 (PF14)
- net PF15: now reaches J11.1 (Pin_1), U2.55 (PF15)
- net PE7: now reaches J14.9 (Pin_9), U2.58 (PE7)
- net PE8: now reaches J14.8 (Pin_8), U2.59 (PE8)
- net PE9: now reaches J14.7 (Pin_7), U2.60 (PE9)
- net PE10: now reaches J14.6 (Pin_6), U2.63 (PE10)
- net PE11: now reaches J14.5 (Pin_5), U2.64 (PE11)
- net PE12: now reaches J14.4 (Pin_4), U2.65 (PE12)
- net PE13: now reaches J14.3 (Pin_3), U2.66 (PE13)
- net PE14: now reaches J14.2 (Pin_2), U2.67 (PE14)
- net PE15: now reaches J14.1 (Pin_1), U2.68 (PE15)
- net PC13: now reaches U2.7 (PC13)
- net PC13: now also J9.11 (Pin_11)
- net PB12: now reaches U2.73 (PB12)
- net PB12: now also J2.15 (Pin_15)
- net PB14: now reaches U2.75 (PB14)
- net PB14: now also J2.16 (Pin_16)
- net PB15: now reaches U2.76 (PB15)
- net PB15: now also J9.1 (Pin_1)
- net PD8: now reaches U2.77 (PD8)
- net PD8: now also J18.3 (Pin_3)
- net PD9: now reaches U2.78 (PD9)
- net PD9: now also J18.4 (Pin_4)
- net PD10: now reaches U2.79 (PD10)
- net PD10: now also J18.5 (Pin_5)
- net PC14: now reaches U2.8 (PC14)
- net PC14: now also J9.12 (Pin_12)
- net PD11: now reaches U2.80 (PD11)
- net PD11: now also J18.6 (Pin_6)
- net PD12: now reaches U2.81 (PD12)
- net PD12: now also J18.7 (Pin_7)
- net PD13: now reaches U2.82 (PD13)
- net PD13: now also J18.8 (Pin_8)
- net PD14: now reaches U2.85 (PD14)
- net PD14: now also J18.9 (Pin_9)
- net PD15: now reaches U2.86 (PD15)
- net PD15: now also J18.10 (Pin_10)
- net PC15: now reaches U2.9 (PC15)
- net PC15: now also J9.13 (Pin_13)
- net PC6: now reaches U2.96 (PC6)
- net PC6: now also J9.8 (Pin_8)
- net PC7: now reaches U2.97 (PC7)
- net PC7: now also J9.9 (Pin_9)
- net PC8: now reaches U2.98 (PC8)
- net PC8: now also J9.10 (Pin_10)
- net RX renamed USART3_TX
- net TX renamed USART3_RX
- new net: J16.A5 (CC1), R2.1
- new net: J16.B5 (CC2), R7.1
- new net: C28.2, C29.1
- no-connect marks 1 -> 60
Other:
- note added: "CL=2*(CL0-Cs)=2*(10-3)=14pF"
- note added: "Decoupling Capacitors"
- note added: "VDDA Filtering"
- note added: "https://www.mouser.com/catalog/specsheets/an10911.pdf"

Commit message: Added LDO power supply
Parts:
- added H1, H2, H3, H4: MountingHole, MountingHole:MountingHole_2.2mm_M2, symbol Mechanical:MountingHole
Other:
- added sheet MCU (MCU.kicad_sch)
- note added: "Use M2-size"
